File: modularFeedbackProcessor/linkedMixer.kicad_sch (KiCad schematic)
At the start: 41 parts, among them Q10 Q_PMOS_GDS, Q11 Q_PMOS_GDS, Q2 Q_NMOS_GDS, Q3 Q_NMOS_GDS, Q4 Q_NMOS_GDS, Q5 Q_NMOS_GDS, Q7 Q_PMOS_GDS, Q8 Q_PMOS_GDS, Q9 Q_PMOS_GDS, U5 LM13700, U6 TL074, U7 LM13700

Commit message: pushing changes
Parts:
- C10: renamed from C11; footprint (none) -> Capacitor_THT:CP_Radial_D5.0mm_P2.50mm
- C6: renamed from C12; footprint (none) -> Capacitor_THT:C_Disc_D4.7mm_W2.5mm_P5.00mm
- C7: renamed from C8; footprint (none) -> Capacitor_THT:CP_Radial_D5.0mm_P2.50mm
- C8: renamed from C10; footprint (none) -> Capacitor_THT:CP_Radial_D5.0mm_P2.50mm
- C9: footprint (none) -> Capacitor_THT:CP_Radial_D5.0mm_P2.50mm
- renumbered D2 to D9, Q4 to Q10, Q9 to Q11, Q5 to Q3, Q7 to Q4, Q10 to Q5, Q2 to Q6, Q11 to Q7, Q3 to Q8, Q8 to Q9, R15 to R39, R17 to R40, R22 to R41, R19 to R42, R23 to R43, R16 to R44, R24 to R45, R31 to R46, R18 to R47, R25 to R48, R32 to R49, R20 to R50, R26 to R51, R21 to R52, R27 to R53, R13 to R54, R14 to R55, R29 to R56, R28 to R57, R30 to R58, RV4 to RV2, RV2 to RV3, RV3 to RV4, U6 to U1, U7 to U5, U5 to U9

Commit message: added all footprints, beginning to work on ERC errors
Parts:
- C10, C7, C8, C9: footprint Capacitor_THT:CP_Radial_D5.0mm_P2.50mm -> Capacitor_SMD:C_0805_2012Metric_Pad1.18x1.45mm_HandSolder
- C6: footprint Capacitor_THT:C_Disc_D4.7mm_W2.5mm_P5.00mm -> Capacitor_SMD:C_0805_2012Metric_Pad1.18x1.45mm_HandSolder
- Q10, Q11, Q3, Q4, Q5, Q6, Q7, Q8, Q9: footprint (none) -> Package_TO_SOT_THT:TO-220-3_Vertical
- R39, R40, R41, R42, R43, R44, R45, R46, R47, R48, R49, R50, R51, R52, R53, R54, R55, R56, R57, R58: footprint (none) -> Resistor_SMD:R_0805_2012Metric_Pad1.20x1.40mm_HandSolder
- RV2, RV3, RV4: footprint (none) -> Potentiometer_THT:Potentiometer_Vishay_T73XW_Horizontal
- U1, U5, U9: footprint (none) -> Package_DIP:DIP-14_W7.62mm_LongPads
Changed lines of the file:
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@@
 			)
 		)
-		(property "Footprint" ""
+		(property "Footprint" "Resistor_SMD:R_0805_2012Metric_Pad1.20x1.40mm_HandSolder"
 			(at 78.232 171.45 90)
 			(hide yes)
@@
 			)
 		)
-		(property "Footprint" ""
+		(property "Footprint" "Resistor_SMD:R_0805_2012Metric_Pad1.20x1.40mm_HandSolder"
 			(at 156.21 128.778 90)
 			(hide yes)
@@
 			)
 		)
-		(property "Footprint" ""
+		(property "Footprint" "Resistor_SMD:R_0805_2012Metric_Pad1.20x1.40mm_HandSolder"
 			(at 70.612 120.65 90)
 			(hide yes)
@@
 			)
 		)
-		(property "Footprint" ""
+		(property "Footprint" "Potentiometer_THT:Potentiometer_Vishay_T73XW_Horizontal"
 			(at 100.33 116.84 0)
 			(hide yes)
@@
 			)
 		)
-		(property "Footprint" ""
+		(property "Footprint" "Resistor_SMD:R_0805_2012Metric_Pad1.20x1.40mm_HandSolder"
 			(at 76.708 101.6 90)
 			(hide yes)
@@
 			)
 		)
-		(property "Footprint" ""
+		(property "Footprint" "Package_TO_SOT_THT:TO-220-3_Vertical"
 			(at 82.55 45.72 0)
 			(hide yes)
@@
 			)
 		)
-		(property "Footprint" ""
+		(property "Footprint" "Resistor_SMD:R_0805_2012Metric_Pad1.20x1.40mm_HandSolder"
 			(at 90.17 61.468 90)
 			(hide yes)
@@
 			)
 		)
-		(property "Footprint" ""
+		(property "Footprint" "Package_DIP:DIP-14_W7.62mm_LongPads"
 			(at 81.28 159.385 0)
 			(hide yes)
@@
 			)
 		)
-		(property "Footprint" ""
+		(property "Footprint" "Resistor_SMD:R_0805_2012Metric_Pad1.20x1.40mm_HandSolder"
 			(at 111.252 116.84 90)
 			(hide yes)
@@
 			)
 		)
-		(property "Footprint" ""
+		(property "Footprint" "Resistor_SMD:R_0805_2012Metric_Pad1.20x1.40mm_HandSolder"
 			(at 64.77 113.538 90)
 			(hide yes)
@@
 			)
 		)
-		(property "Footprint" ""
+		(property "Footprint" "Resistor_SMD:R_0805_2012Metric_Pad1.20x1.40mm_HandSolder"
 			(at 76.708 152.4 90)
 			(hide yes)
@@
 			)
 		)
-		(property "Footprint" ""
+		(property "Footprint" "Resistor_SMD:R_0805_2012Metric_Pad1.20x1.40mm_HandSolder"
 			(at 156.21 136.398 90)
 			(hide yes)
@@
 			)
 		)
-		(property "Footprint" "Capacitor_THT:C_Disc_D4.7mm_W2.5mm_P5.00mm"
+		(property "Footprint" "Capacitor_SMD:C_0805_2012Metric_Pad1.18x1.45mm_HandSolder"
 			(at 50.8 58.7248 0)
 			(hide yes)
@@
 			)
 		)
-		(property "Footprint" ""
+		(property "Footprint" "Package_TO_SOT_THT:TO-220-3_Vertical"
 			(at 77.47 39.37 0)
 			(hide yes)
@@
 			)
 		)
-		(property "Footprint" ""
+		(property "Footprint" "Package_TO_SOT_THT:TO-220-3_Vertical"
 			(at 87.63 69.85 0)
 			(hide yes)
@@
 			)
 		)
-		(property "Footprint" ""
+		(property "Footprint" "Resistor_SMD:R_0805_2012Metric_Pad1.20x1.40mm_HandSolder"
 			(at 137.922 74.93 90)
 			(hide yes)
@@
 			)
 		)
-		(property "Footprint" ""
+		(property "Footprint" "Resistor_SMD:R_0805_2012Metric_Pad1.20x1.40mm_HandSolder"
 			(at 29.21 36.068 90)
 			(hide yes)
@@
 			)
 		)
-		(property "Footprint" ""
+		(property "Footprint" "Package_DIP:DIP-14_W7.62mm_LongPads"
 			(at 101.6 159.385 0)
 			(hide yes)
@@
 			)
 		)
-		(property "Footprint" ""
+		(property "Footprint" "Package_DIP:DIP-14_W7.62mm_LongPads"
 			(at 101.6 108.585 0)
 			(hide yes)
@@
 			)
 		)
-		(property "Footprint" ""
+		(property "Footprint" "Potentiometer_THT:Potentiometer_Vishay_T73XW_Horizontal"
 			(at 39.37 34.29 0)
 			(hide yes)
@@
 			)
 		)
-		(property "Footprint" ""
+		(property "Footprint" "Resistor_SMD:R_0805_2012Metric_Pad1.20x1.40mm_HandSolder"
 			(at 121.412 116.84 90)
 			(hide yes)
@@
 			)
 		)
-		(property "Footprint" ""
+		(property "Footprint" "Resistor_SMD:R_0805_2012Metric_Pad1.20x1.40mm_HandSolder"
 			(at 111.252 167.64 90)
 			(hide yes)
@@
 			)
 		)
-		(property "Footprint" ""
+		(property "Footprint" "Package_DIP:DIP-14_W7.62mm_LongPads"
 			(at 55.88 39.37 0)
 			(hide yes)
@@
 			)
 		)
-		(property "Footprint" ""
+		(property "Footprint" "Package_TO_SOT_THT:TO-220-3_Vertical"
 			(at 105.41 45.72 0)
 			(hide yes)
@@
 			)
 		)
-		(property "Footprint" "Capacitor_THT:CP_Radial_D5.0mm_P2.50mm"
+		(property "Footprint" "Capacitor_SMD:C_0805_2012Metric_Pad1.18x1.45mm_HandSolder"
 			(at 58.42 161.5948 0)
 			(hide yes)
@@
 			)
 		)
-		(property "Footprint" ""
+		(property "Footprint" "Resistor_SMD:R_0805_2012Metric_Pad1.20x1.40mm_HandSolder"
 			(at 64.77 164.338 90)
 			(hide yes)
@@
 			)
 		)
-		(property "Footprint" ""
+		(property "Footprint" "Package_TO_SOT_THT:TO-220-3_Vertical"
 			(at 100.33 62.23 0)
 			(hide yes)
@@
 			)
 		)
-		(property "Footprint" ""
+		(property "Footprint" "Package_DIP:DIP-14_W7.62mm_LongPads"
 			(at 171.45 139.7 0)
 			(hide yes)
@@
 			)
 		)
-		(property "Footprint" ""
+		(property "Footprint" "Package_DIP:DIP-14_W7.62mm_LongPads"
 			(at 81.28 108.585 0)
 			(hide yes)
@@
 			)
 		)
-		(property "Footprint" ""
+		(property "Footprint" "Package_TO_SOT_THT:TO-220-3_Vertical"
 			(at 119.38 77.47 0)
 			(hide yes)
@@
 			)
 		)
-		(property "Footprint" ""
+		(property "Footprint" "Resistor_SMD:R_0805_2012Metric_Pad1.20x1.40mm_HandSolder"
 			(at 123.952 74.93 90)
 			(hide yes)
@@
 			)
 		)
-		(property "Footprint" ""
+		(property "Footprint" "Package_DIP:DIP-14_W7.62mm_LongPads"
 			(at 53.34 69.85 0)
 			(hide yes)
@@
 			)
 		)
-		(property "Footprint" ""
+		(property "Footprint" "Potentiometer_THT:Potentiometer_Vishay_T73XW_Horizontal"
 			(at 100.33 167.64 0)
 			(hide yes)
@@
 			)
 		)
-		(property "Footprint" ""
+		(property "Footprint" "Package_TO_SOT_THT:TO-220-3_Vertical"
 			(at 105.41 77.47 0)
 			(hide yes)
@@
 			)
 		)
-		(property "Footprint" "Capacitor_THT:CP_Radial_D5.0mm_P2.50mm"
+		(property "Footprint" "Capacitor_SMD:C_0805_2012Metric_Pad1.18x1.45mm_HandSolder"
 			(at 58.42 110.7948 0)
 			(hide yes)
@@
 			)
 		)
-		(property "Footprint" ""
+		(property "Footprint" "Package_DIP:DIP-14_W7.62mm_LongPads"
 			(at 248.92 36.195 0)
 			(hide yes)
@@
 			)
 		)
-		(property "Footprint" ""
+		(property "Footprint" "Resistor_SMD:R_0805_2012Metric_Pad1.20x1.40mm_HandSolder"
 			(at 172.72 131.318 90)
 			(hide yes)
@@
 			)
 		)
-		(property "Footprint" "Capacitor_THT:CP_Radial_D5.0mm_P2.50mm"
+		(property "Footprint" "Capacitor_SMD:C_0805_2012Metric_Pad1.18x1.45mm_HandSolder"
 			(at 121.92 161.5948 0)
 			(hide yes)
@@
 			)
 		)
-		(property "Footprint" ""
+		(property "Footprint" "Package_TO_SOT_THT:TO-220-3_Vertical"
 			(at 82.55 77.47 0)
 			(hide yes)
@@
 			)
 		)
-		(property "Footprint" ""
+		(property "Footprint" "Resistor_SMD:R_0805_2012Metric_Pad1.20x1.40mm_HandSolder"
 			(at 70.612 171.45 90)
 			(hide yes)
@@
 			)
 		)
-		(property "Footprint" ""
+		(property "Footprint" "Resistor_SMD:R_0805_2012Metric_Pad1.20x1.40mm_HandSolder"
 			(at 78.232 120.65 90)
 			(hide yes)
@@
 			)
 		)
-		(property "Footprint" "Capacitor_THT:CP_Radial_D5.0mm_P2.50mm"
+		(property "Footprint" "Capacitor_SMD:C_0805_2012Metric_Pad1.18x1.45mm_HandSolder"
 			(at 121.92 110.7948 0)
 			(hide yes)
@@
 			)
 		)
-		(property "Footprint" ""
+		(property "Footprint" "Resistor_SMD:R_0805_2012Metric_Pad1.20x1.40mm_HandSolder"
 			(at 121.412 167.64 90)
 			(hide yes)
@@
 			)
 		)
-		(property "Footprint" ""
+		(property "Footprint" "Resistor_SMD:R_0805_2012Metric_Pad1.20x1.40mm_HandSolder"
 			(at 80.01 61.468 90)
 			(hide yes)
@@
 			)
 		)
-		(property "Footprint" ""
+		(property "Footprint" "Package_TO_SOT_THT:TO-220-3_Vertical"
 			(at 123.19 62.23 0)
 			(hide yes)

Commit message: lots of friggin progress. finished footprint work, and have just finished grouping. Now I will start to connect each group internally.
Parts:
- removed U5: LM13700, Package_DIP:DIP-14_W7.62mm_LongPads, symbol Amplifier_Operational:LM13700
- added C20, C21, C31, C33: 100n, Capacitor_SMD:C_0805_2012Metric_Pad1.18x1.45mm_HandSolder, symbol Device:C
- added TP12: MixTune1, PCM_4ms_TestPoint:TestPoint_Pad_06, symbol PCM_4ms_Connector:TestPoint_Small
- added TP14: MixerV1, PCM_4ms_TestPoint:TestPoint_Pad_06, symbol PCM_4ms_Connector:TestPoint_Small
- added TP16: MixerV2, PCM_4ms_TestPoint:TestPoint_Pad_06, symbol PCM_4ms_Connector:TestPoint_Small
- added TP18: MixerV1o, PCM_4ms_TestPoint:TestPoint_Pad_06, symbol PCM_4ms_Connector:TestPoint_Small
- added TP20: MixerV2o, PCM_4ms_TestPoint:TestPoint_Pad_06, symbol PCM_4ms_Connector:TestPoint_Small
- added TP22: MixerOut, PCM_4ms_TestPoint:TestPoint_Pad_06, symbol PCM_4ms_Connector:TestPoint_Small
- added unit 1 of U1
- added unit 5 of U1
- U8: renamed from U9; footprint Package_DIP:DIP-14_W7.62mm_LongPads -> Package_DIP:DIP-16_W7.62mm_LongPads
- renumbered D9 to D8, Q11 to Q10, Q3 to Q2, Q4 to Q3, Q5 to Q4, Q6 to Q5, Q7 to Q6, Q8 to Q7, Q9 to Q8, Q10 to Q9, R39 to R41, R40 to R42, R41 to R43, R42 to R44, R43 to R45, R44 to R46, R45 to R47, R46 to R48, R47 to R49, R48 to R50, R49 to R51, R50 to R52, R51 to R53, R52 to R54, R53 to R55, R54 to R56, R55 to R57, R56 to R58, R57 to R59, R58 to R60, RV2 to RV12, RV3 to RV13, RV4 to RV14
Connections:
- net +12V: now also U8.11 (V+), C20.1, C33.1, U1.4 (V+)
- net -12V: now also U8.6 (V-), C21.2, C31.2, U1.11 (V-)
- net GND: now also C20.2, C21.1, C31.1, C33.2, U1.3 (+)
- net V_{in1}: now also TP14.1
- net V_{in2}: now also TP16.1
- net V_{out}: now also TP22.1, U1.1; no longer U1.14
- net at C9.2, R54.1, R58.1: now also TP18.1
- net at R58.2, R59.2, R60.1: now also U1.2 (-); no longer U1.13 (-)
- net at C10.2, R55.1, R59.1: now also TP20.1
- net at Q2.3 (S), RV12.3, U1.6 (-): now also TP12.1
- new net: U1.13 (-), U1.14
Other:
- note added: "connecting unused op amp as per TI's recommendation"
