File: modularFeedbackProcessor/Mixer.kicad_sch (KiCad schematic)
At the start: 50 parts, among them Q10 Q_PMOS_GDS, Q2 Q_NMOS_GDS, Q3 Q_PMOS_GDS, Q4 Q_PMOS_GDS, Q5 Q_NMOS_GDS, Q6 Q_PMOS_GDS, Q7 Q_NMOS_GDS, Q8 Q_PMOS_GDS, Q9 Q_NMOS_GDS, U1 TL074, U8 LM13700

Commit message: save before i mess something up
Parts:
- removed C10, C7, C8, C9: 2.2u, Capacitor_SMD:C_0805_2012Metric_Pad1.18x1.45mm_HandSolder, symbol Device:C
- removed C31, C33: 100n, Capacitor_SMD:C_0805_2012Metric_Pad1.18x1.45mm_HandSolder, symbol Device:C
- removed C6: 1n, Capacitor_SMD:C_0805_2012Metric_Pad1.18x1.45mm_HandSolder, symbol Device:C
- removed D8: 1N4148, Diode_THT:D_DO-35_SOD27_P7.62mm_Horizontal, symbol Diode:1N4148
- removed R41, R42, R43: 18k, Resistor_SMD:R_0805_2012Metric_Pad1.20x1.40mm_HandSolder, symbol Device:R
- removed TP18: MixerV1o, PCM_4ms_TestPoint:TestPoint_Pad_06, symbol PCM_4ms_Connector:TestPoint_Small
- removed TP20: MixerV2o, PCM_4ms_TestPoint:TestPoint_Pad_06, symbol PCM_4ms_Connector:TestPoint_Small
- removed TP22: MixerOut, PCM_4ms_TestPoint:TestPoint_Pad_06, symbol PCM_4ms_Connector:TestPoint_Small
- removed U1: TL074, Package_DIP:DIP-14_W7.62mm_LongPads, symbol Amplifier_Operational:TL074
- added C17: 1n, Capacitor_SMD:C_0805_2012Metric_Pad1.18x1.45mm_HandSolder, symbol Device:C
- added C18, C19: 2.2u, Capacitor_SMD:C_0805_2012Metric_Pad1.18x1.45mm_HandSolder, symbol Device:C
- added C22, C23, C24, C25: 100n, Capacitor_SMD:C_0805_2012Metric_Pad1.18x1.45mm_HandSolder, symbol Device:C
- added D11: 1N4148, Diode_THT:D_DO-35_SOD27_P7.62mm_Horizontal, symbol Diode:1N4148
- added R61, R62, R63: 1k, Resistor_SMD:R_0805_2012Metric_Pad1.20x1.40mm_HandSolder, symbol Device:R
- added TP13: MixerV2, PCM_4ms_TestPoint:TestPoint_Pad_06, symbol PCM_4ms_Connector:TestPoint_Small
- added TP15: MixerV1o, PCM_4ms_TestPoint:TestPoint_Pad_06, symbol PCM_4ms_Connector:TestPoint_Small
- added TP17: MixerOut, PCM_4ms_TestPoint:TestPoint_Pad_06, symbol PCM_4ms_Connector:TestPoint_Small
- added U7: TL074, Package_DIP:DIP-14_W7.62mm_LongPads, symbol Amplifier_Operational:TL074
- C20, C21: value 100n -> 2.2u
- R44, R45: value 560 -> 18k
- R46: value 12k -> 18k
- R47: value 12k -> 560
- R48: value 33k -> 560
- R49, R50: value 560 -> 12k
- R51: value 1k -> 33k
- R52, R53: value 5.6k -> 560
- R54: value 100k -> 1k
- R55: value 100k -> 5.6k
- R56: value 6.8k -> 5.6k
- R57: value 6.8k -> 100k
- R58: value 1k -> 100k
- R59, R60: value 1k -> 6.8k
- TP12: value MixTune1 -> MixerV1
- TP14: value MixerV1 -> MixTune1
- TP16: value MixerV2 -> MixerV2o
Connections:
- net +12V: now also R49.2, R50.2, C22.1, C24.1, U7.4 (V+); no longer C20.1, R46.2, R47.2
- net -12V: now also R44.1, R55.2, R56.2, C23.2, C25.2, U7.11 (V-); no longer C21.2, R52.2, R53.2
- net GND: now also R47.2, R48.2, R52.2, R53.2, R57.2, R58.2, C22.2, C23.1, C24.2, C25.1, U7.10 (+), U7.12 (+), U7.3 (+), U7.5 (+); no longer C20.2, C21.1, R44.2, R45.2, R49.2, R50.2, R51.2, R55.2
- net Iout1: now also R60.2; no longer R57.2
- net Iout2: now also R59.2; no longer R56.2
- net V_{ctrl}: now also R51.1, C17.2, D11.1 (K), U7.9 (-); no longer R48.1
- net V_{in1}: now also TP12.1, C18.1; no longer TP14.1
- net V_{in2}: now also C19.1, TP13.1; no longer TP16.1
- net V_{out}: now also R63.2, TP17.1, U7.1; no longer R60.2
- net at R53.1: now also U8.4 (-); no longer U8.8
- net at U8.14 (+): now also R45.2, R47.1; no longer R44.1
- net at U8.2 (DIODE_BIAS): now also R50.1; no longer R47.1
- net at Q2.1 (G): now also U7.7
- net at Q2.3 (S), RV12.3: now also TP14.1, U7.6 (-); no longer TP12.1
- net at R55.1: now also C20.1, U8.9; no longer R59.1
- net at R49.1: now also U8.15 (DIODE_BIAS); no longer U8.13 (-)
- net at R46.1: now also C19.2; no longer U8.15 (DIODE_BIAS)
- net at R54.1: now also Q3.3 (S), R51.2; no longer R58.1
- net at Q6.2 (D), Q9.2 (D): now also R59.1; no longer R56.1
- net at R57.1: now also C20.2, R61.1, TP15.1; no longer Q10.2 (D)
- net at R52.1: now also U8.13 (-); no longer U8.9
- net at Q3.1 (G): now also C17.1, D11.2 (A), U7.8
- net at RV12.1, RV12.2: now also R44.2
- net at U8.3 (+): now also R46.2, R48.1; no longer R45.1
- new net: R61.2, R62.2, R63.1, U7.2 (-)
- new net: U7.13 (-), U7.14
- new net: C18.2, R45.1
- new net: C21.2, R58.1, R62.1, TP16.1
- new net: Q10.2 (D), R60.1
- new net: C21.1, R56.1, U8.8
