File: modularFeedbackProcessor/MFP.kicad_blocks/Mixer.kicad_block/Mixer.kicad_sch (KiCad schematic)
At the start: 0 parts

Commit message: Update: did not destroy everything
Parts:
- added C17: 1n, Capacitor_SMD:C_0805_2012Metric_Pad1.18x1.45mm_HandSolder, symbol Device:C
- added C18, C19, C20, C21: 2.2u, Capacitor_SMD:C_0805_2012Metric_Pad1.18x1.45mm_HandSolder, symbol Device:C
- added C22, C23, C24, C25: 100n, Capacitor_SMD:C_0805_2012Metric_Pad1.18x1.45mm_HandSolder, symbol Device:C
- added D11: 1N4148, Diode_THT:D_DO-35_SOD27_P7.62mm_Horizontal, symbol Diode:1N4148
- added Q10, Q3, Q4, Q6, Q8: Q_PMOS_GDS, Package_TO_SOT_THT:TO-220-3_Vertical, symbol Transistor_FET:Q_PMOS_GDS
- added Q2, Q5, Q7, Q9: Q_NMOS_GDS, Package_TO_SOT_THT:TO-220-3_Vertical, symbol Transistor_FET:Q_NMOS_GDS
- added R44, R45, R46: 18k, Resistor_SMD:R_0805_2012Metric_Pad1.20x1.40mm_HandSolder, symbol Device:R
- added R47, R48, R52, R53: 560, Resistor_SMD:R_0805_2012Metric_Pad1.20x1.40mm_HandSolder, symbol Device:R
- added R49, R50: 12k, Resistor_SMD:R_0805_2012Metric_Pad1.20x1.40mm_HandSolder, symbol Device:R
- added R51: 33k, Resistor_SMD:R_0805_2012Metric_Pad1.20x1.40mm_HandSolder, symbol Device:R
- added R54, R61, R62, R63: 1k, Resistor_SMD:R_0805_2012Metric_Pad1.20x1.40mm_HandSolder, symbol Device:R
- added R55, R56: 5.6k, Resistor_SMD:R_0805_2012Metric_Pad1.20x1.40mm_HandSolder, symbol Device:R
- added R57, R58: 100k, Resistor_SMD:R_0805_2012Metric_Pad1.20x1.40mm_HandSolder, symbol Device:R
- added R59, R60: 6.8k, Resistor_SMD:R_0805_2012Metric_Pad1.20x1.40mm_HandSolder, symbol Device:R
- added RV12: 10k, Potentiometer_THT:Potentiometer_Vishay_T73XW_Horizontal, symbol Device:R_Potentiometer_Trim
- added RV13, RV14: 50k, Potentiometer_THT:Potentiometer_Vishay_T73XW_Horizontal, symbol Device:R_Potentiometer_Trim
- added TP12: MixerV1, PCM_4ms_TestPoint:TestPoint_Pad_06, symbol PCM_4ms_Connector:TestPoint_Small
- added TP13: MixerV2, PCM_4ms_TestPoint:TestPoint_Pad_06, symbol PCM_4ms_Connector:TestPoint_Small
- added TP14: MixTune1, PCM_4ms_TestPoint:TestPoint_Pad_06, symbol PCM_4ms_Connector:TestPoint_Small
- added TP15: MixerV1o, PCM_4ms_TestPoint:TestPoint_Pad_06, symbol PCM_4ms_Connector:TestPoint_Small
- added TP16: MixerV2o, PCM_4ms_TestPoint:TestPoint_Pad_06, symbol PCM_4ms_Connector:TestPoint_Small
- added TP17: MixerOut, PCM_4ms_TestPoint:TestPoint_Pad_06, symbol PCM_4ms_Connector:TestPoint_Small
- added U7: TL074, Package_DIP:DIP-14_W7.62mm_LongPads, symbol Amplifier_Operational:TL074
- added U8: LM13700, Package_DIP:DIP-16_W7.62mm_LongPads, symbol Amplifier_Operational:LM13700
Connections:
- new net: R53.1, U8.4 (-)
- new net: C20.2, R57.1, R61.1, TP15.1
- new net: R61.2, R62.2, R63.1, U7.2 (-)
- new net: R45.2, R47.1, U8.14 (+)
- new net: RV13.1, U8.10, U8.12
- new net: R49.1, U8.15 (DIODE_BIAS)
- new net: Q2.2 (D), Q4.1 (G), Q4.2 (D), Q6.1 (G)
- new net: U7.13 (-), U7.14
- new net: Q3.3 (S), R51.2, R54.1
- new net: R50.1, U8.2 (DIODE_BIAS)
- new net: R46.2, R48.1, U8.3 (+)
- new net: RV14.1, U8.5, U8.7
- new net: Q2.3 (S), RV12.3, TP14.1, U7.6 (-)
- new net: C20.1, R55.1, U8.9
- new net: C18.2, R45.1
- new net: C21.2, R58.1, R62.1, TP16.1
- new net: C17.1, D11.2 (A), Q3.1 (G), U7.8
- new net: Q2.1 (G), U7.7
- new net: Q3.2 (D), Q5.1 (G), Q5.2 (D), Q7.1 (G), Q9.1 (G)
- new net: Q10.2 (D), R60.1
- new net: R44.2, RV12.1, RV12.2
- new net: C21.1, R56.1, U8.8
- new net: Q6.2 (D), Q9.2 (D), R59.1
- new net: C19.2, R46.1
- new net: Q10.1 (G), Q7.2 (D), Q8.1 (G), Q8.2 (D)
- new net: R52.1, U8.13 (-)
- new net +12V: C22.1, C24.1, Q10.3 (S), Q4.3 (S), Q6.3 (S), Q8.3 (S), R49.2, R50.2, U7.4 (V+), U8.11 (V+)
- new net -12V: C23.2, C25.2, Q5.3 (S), Q7.3 (S), Q9.3 (S), R44.1, R55.2, R56.2, U7.11 (V-), U8.6 (V-)
- new net GND: C22.2, C23.1, C24.2, C25.1, R47.2, R48.2, R52.2, R53.2, R54.2, R57.2, R58.2, RV13.2, RV13.3, RV14.2, RV14.3, U7.10 (+), U7.12 (+), U7.3 (+), U7.5 (+)
- new net Iout1: R60.2, U8.1
- new net Iout2: R59.2, U8.16
- new net V_{ctrl}: C17.2, D11.1 (K), R51.1, U7.9 (-)
- new net V_{in1}: C18.1, TP12.1
- new net V_{in2}: C19.1, TP13.1
- new net V_{out}: R63.2, TP17.1, U7.1
Other:
- removed sheet DryWet Mixer
- note added: "0-5V should be connected with 330k resistors"
- note added: "connecting unused op amp as per TI's recommendation"
- note added: "tune for unity gain"
- note added: "tune to 24k total"
